File: PCF8574AN.sch (KiCad schematic (older format))
At the start: 8 parts, among them J1 Conn_01x04, J2 Conn_01x03, J3 Conn_01x10, J4 Conn_01x04, U1 PCF8574

Commit message: Migrate project to new Kicad version. Adding headers for change address of chip PCF8574.
Parts:
- removed J1, J4: Conn_01x04, Pin_Headers:Pin_Header_Straight_1x04_Pitch2.54mm, symbol Conn_01x04
- removed J2: Conn_01x03, Pin_Headers:Pin_Header_Straight_1x03_Pitch2.54mm, symbol Conn_01x03
- removed J3: Conn_01x10, Pin_Headers:Pin_Header_Straight_1x10_Pitch2.54mm, symbol Conn_01x10
- removed R1, R2: 2.2k, Resistors_SMD:R_1206, symbol R
- removed R3: R, Resistors_SMD:R_1206, symbol R
- added J1, J4: Conn_01x04_Male, Connector_PinHeader_2.54mm:PinHeader_1x04_P2.54mm_Vertical, symbol Connector:Conn_01x04_Male
- added J2, J5, J6: Conn_01x03_Male, Connector_PinHeader_2.54mm:PinHeader_1x03_P2.54mm_Vertical, symbol Connector:Conn_01x03_Male
- added J3: Conn_01x10_Male, Connector_PinHeader_2.54mm:PinHeader_1x10_P2.54mm_Vertical, symbol Connector:Conn_01x10_Male
- added R1, R2, R3, R4, R5, R6: R, Resistor_SMD:R_1206_3216Metric, symbol Device:R
- U1: footprint Housings_DIP:DIP-16_W7.62mm_LongPads -> Package_DIP:DIP-16_W7.62mm_LongPads; symbol PCF8574 -> PCF8574AN-rescue:PCF8574
Connections:
- wire segments 48 -> 88
Other:
- moved on the sheet: U1
